File: hardware/termination.kicad_pcb (KiCad board)
At the start: 2 copper layers, 20.3 x 11.4 mm, 9 parts, among them P1 CONN_01X04, P2 CONN_01X04

Commit message: o Make fab generation work for multiple targets independently o Use smaller font on Termination board for git version.
Other:
- board text added: "%%gitversion%%"
- board text added: "flaschen-taschen Termination"
- board text removed: "flaschen-taschen Termination %%gitversion%%"
Changed lines of the file:
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@@
   (general
     (links 17)
-    (no_connects 3)
-    (area 147.244999 95.174999 167.715001 106.755001)
+    (no_connects 0)
+    (area 144.116667 90.93 174.070001 107.147)
     (thickness 1.6)
-    (drawings 9)
+    (drawings 10)
     (tracks 35)
     (zones 0)
@@
     )
   )
+  (gr_text %%gitversion%% (at 156.337 98.425 180) (layer B.SilkS)
+    (effects (font (size 0.7 0.6) (thickness 0.1)) (justify mirror))
+  )
   (gr_text "GND\n" (at 164.465 97.155 180) (layer B.SilkS)
     (effects (font (size 1 1) (thickness 0.15)) (justify left mirror))
@@
     (effects (font (size 1 1) (thickness 0.15)) (justify left mirror))
   )
-  (gr_text "flaschen-taschen\nTermination\n\n%%gitversion%%" (at 156.337 100.965 180) (layer B.SilkS)
+  (gr_text "flaschen-taschen\nTermination\n" (at 156.337 102.235 180) (layer B.SilkS)
     (effects (font (size 0.8 0.8) (thickness 0.15)) (justify mirror))
   )
